File: board_shematic/controller board v2 with better symbols/controller board v2/controller board v2.kicad_sch (KiCad schematic)
At the start: 18 parts, among them J1 Conn_01x03_Pin, J2 Conn_01x03_Pin, J3 Conn_01x03_Pin, J4 Conn_01x05_Pin, J5 Conn_01x07_Pin, SW1 SW_Push, SW2 SW_Push, SW3 SW_Push, SW4 SW_Push, SW5 SW_Push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

Commit message: minor edits to pcb, end of night
Parts:
- U1, U2: footprint SparkFun-Electromechanical:XDCR_COM-09032 -> joystick:XDCR_COM-09032
Changed lines of the file:
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@@
       (effects (font (size 1.27 1.27)) (justify left))
     )
-    (property "Footprint" "SparkFun-Electromechanical:XDCR_COM-09032" (at 286.512 182.88 0)
+    (property "Footprint" "joystick:XDCR_COM-09032" (at 286.512 182.88 0)
       (effects (font (size 0.508 0.508)) hide)
     )
@@
       (effects (font (size 1.27 1.27)) (justify left))
     )
-    (property "Footprint" "SparkFun-Electromechanical:XDCR_COM-09032" (at 286.512 137.16 0)
+    (property "Footprint" "joystick:XDCR_COM-09032" (at 286.512 137.16 0)
       (effects (font (size 0.508 0.508)) hide)
     )
